File: flypanels.sch (KiCad schematic (older format))
At the start: 1 part

Commit message: board routed.
Parts:
- added C1, C2: 0.1uF, symbol C
- added MATRIX1: LED_8X8, symbol LED_8X8
- added P1, P2: CONN_8, symbol CONN_8
- added R1, R2, R3, R4, R5, R6, R7, R8: 82, symbol R
- added R9: 10K, symbol R
- added U1: ULN2804A, symbol ULN2804A
- added X1: CER_RESO, symbol CER_RESO
- gave numbers to parts that had none: 1
Connections:
- wire segments 9 -> 99
- no-connect marks 0 -> 6
Other:
- note added: "BOTTOM"
- note added: "TOP"
- moved on the sheet: IC1
